File: eagle_design/Analog.sch (EAGLE design)
At the start: 18 parts, among them K1 G5LE, K2 G5LE, K3 G5LE

Commit message: Did some more PCB design and added some datasheets
Parts:
- removed D4, D5, D6, D7: 1N4004, diode:1N4004
- added B1: RECTIFIER-S80, rectifier:RECTIFIER-S80
- added SV3, SV4: (no value), con-lstb:MA05-1
Connections:
- removed net 5V-: C1.-, C2.-, D6.A, D7.A, D8.A, VREG-3.3G$1.GND, VREG-5.GND, VREG-5.ON_N
- new net G: K32.S, SV4.1
- new net N$6: K12.O
- new net N$7: K22.O
- new net N$8: K32.O
- new net W: K12.S, SV4.3
- new net Y: K22.S, SV4.2
- net 3.3+: now also SV3.5
- net AC: now also SV3.2
- net FAN: now also SV3.1
- net GND: now also B1.-, C1.-, C2.-, D8.A, SV3.4, VREG-3.3G$1.GND, VREG-5.GND, VREG-5.ON_N
- net HEAT: now also SV3.3
- net N$1: now also B1.+; no longer D4.C, D5.C
- net VAC+: now also B1.AC1, K12.P, K22.P, K32.P, SV4.5; no longer D5.A, D7.C
- net VAC-: now also SV4.4; no longer D4.A, D6.C, K12.O, K12.P, K22.O, K22.P, K32.O, K32.P
