File: eagle_design/Relays.sch (EAGLE design)
At the start: 13 parts, among them K1 G5LE, K2 G5LE, K3 G5LE

Commit message: made boards smaller
Parts:
- removed U$1, U$2: SCREWTERMINAL-2, SparkFun-Connectors:SCREWTERMINAL-2
- removed U$3: SCREWTERMINAL-3, SparkFun-Connectors:SCREWTERMINAL-3
- added U$4, U$5: OSTTC020162, TylersLib:OSTTC020162
- added U$6: OSTTC030162, TylersLib:OSTTC030162
Connections:
- net FIVE+: now also U$5.1; no longer U$1.2
- net G: now also U$6.1; no longer U$3.1
- net GND: now also U$5.2; no longer U$1.1
- net VAC+: now also U$4.1; no longer U$2.2
- net VAC-: now also U$4.2; no longer U$2.1
- net W: now also U$6.3; no longer U$3.3
- net Y: now also U$6.2; no longer U$3.2
Changed lines of the file:
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@@
 <part name="GND6" library="supply1" deviceset="GND" device=""/>
 <part name="GND7" library="supply1" deviceset="GND" device=""/>
-<part name="U$1" library="SparkFun-Connectors" deviceset="SCREWTERMINAL-2" device=""/>
 <part name="SV1" library="con-lstb" deviceset="MA03-1" device=""/>
-<part name="U$2" library="SparkFun-Connectors" deviceset="SCREWTERMINAL-2" device=""/>
-<part name="U$3" library="SparkFun-Connectors" deviceset="SCREWTERMINAL-3" device=""/>
+<part name="U$4" library="TylersLib" deviceset="OSTTC020162" device=""/>
+<part name="U$5" library="TylersLib" deviceset="OSTTC020162" device=""/>
+<part name="U$6" library="TylersLib" deviceset="OSTTC030162" device=""/>
 </parts>
 <sheets>
@@
 <instance part="GND6" gate="1" x="30.48" y="0"/>
 <instance part="GND7" gate="1" x="10.16" y="0"/>
-<instance part="U$1" gate="G$1" x="7.62" y="35.56" rot="R90"/>
 <instance part="SV1" gate="G$1" x="25.4" y="40.64"/>
-<instance part="U$2" gate="G$1" x="50.8" y="35.56" rot="R90"/>
-<instance part="U$3" gate="G$1" x="68.58" y="33.02" rot="R90"/>
+<instance part="U$4" gate="G$1" x="45.72" y="35.56"/>
+<instance part="U$5" gate="G$1" x="2.54" y="35.56"/>
+<instance part="U$6" gate="G$1" x="68.58" y="33.02"/>
 </instances>
 <busses>
@@
 </segment>
 <segment>
-<pinref part="U$1" gate="G$1" pin="1"/>
 <wire x1="12.7" y1="38.1" x2="15.24" y2="38.1" width="0.1524" layer="91"/>
 <junction x="15.24" y="38.1"/>
 <label x="10.16" y="38.1" size="1.778" layer="95"/>
+<pinref part="U$5" gate="G$1" pin="2"/>
 </segment>
 </net>
@@
 </segment>
 <segment>
-<pinref part="U$2" gate="G$1" pin="2"/>
 <wire x1="55.88" y1="40.64" x2="58.42" y2="40.64" width="0.1524" layer="91"/>
 <junction x="58.42" y="40.64"/>
 <label x="53.34" y="40.64" size="1.778" layer="95"/>
+<pinref part="U$4" gate="G$1" pin="1"/>
 </segment>
 </net>
@@
 </segment>
 <segment>
-<pinref part="U$1" gate="G$1" pin="2"/>
 <wire x1="12.7" y1="40.64" x2="15.24" y2="40.64" width="0.1524" layer="91"/>
 <junction x="15.24" y="40.64"/>
 <label x="10.16" y="40.64" size="1.778" layer="95"/>
+<pinref part="U$5" gate="G$1" pin="1"/>
 </segment>
 </net>
@@
 </segment>
 <segment>
-<pinref part="U$3" gate="G$1" pin="3"/>
-<wire x1="73.66" y1="40.64" x2="76.2" y2="40.64" width="0.1524" layer="91"/>
-<junction x="76.2" y="40.64"/>
-<label x="73.66" y="40.64" size="1.778" layer="95"/>
+<pinref part="U$6" gate="G$1" pin="3"/>
+<wire x1="73.66" y1="35.56" x2="76.2" y2="35.56" width="0.1524" layer="91"/>
+<junction x="76.2" y="35.56"/>
+<label x="73.66" y="35.56" size="1.778" layer="95"/>
 </segment>
 </net>
@@
 </segment>
 <segment>
-<pinref part="U$3" gate="G$1" pin="2"/>
 <wire x1="73.66" y1="38.1" x2="76.2" y2="38.1" width="0.1524" layer="91"/>
 <junction x="76.2" y="38.1"/>
 <label x="73.66" y="38.1" size="1.778" layer="95"/>
+<pinref part="U$6" gate="G$1" pin="2"/>
 </segment>
 </net>
@@
 </segment>
 <segment>
-<pinref part="U$3" gate="G$1" pin="1"/>
-<wire x1="73.66" y1="35.56" x2="76.2" y2="35.56" width="0.1524" layer="91"/>
-<junction x="76.2" y="35.56"/>
-<label x="73.66" y="35.56" size="1.778" layer="95"/>
+<pinref part="U$6" gate="G$1" pin="1"/>
+<wire x1="73.66" y1="40.64" x2="76.2" y2="40.64" width="0.1524" layer="91"/>
+<junction x="76.2" y="40.64"/>
+<label x="73.66" y="40.64" size="1.778" layer="95"/>
 </segment>
 </net>
@@
 <net name="VAC-" class="0">
 <segment>
-<pinref part="U$2" gate="G$1" pin="1"/>
 <wire x1="55.88" y1="38.1" x2="58.42" y2="38.1" width="0.1524" layer="91"/>
 <junction x="58.42" y="38.1"/>
 <label x="53.34" y="38.1" size="1.778" layer="95"/>
-</segment>
-</net>
+<pinref part="U$4" gate="G$1" pin="2"/>
+</segment>
+</net>

Commit message: Cleaned up boards and added script to gen gerbers
Changed lines of the file:
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@@
 <wire x1="30.48" y1="22.86" x2="30.48" y2="25.4" width="0.1524" layer="91"/>
 <junction x="30.48" y="25.4"/>
+<junction x="30.48" y="22.86"/>
 </segment>
 <segment>
@@
 <wire x1="10.16" y1="22.86" x2="10.16" y2="25.4" width="0.1524" layer="91"/>
 <junction x="10.16" y="25.4"/>
+<junction x="10.16" y="22.86"/>
 </segment>
 <segment>
@@
 <wire x1="50.8" y1="22.86" x2="50.8" y2="25.4" width="0.1524" layer="91"/>
 <junction x="50.8" y="25.4"/>
+<junction x="50.8" y="22.86"/>
 </segment>
 <segment>
