File: eagle_design/Control.sch (EAGLE design)
At the start: 2 parts

Commit message: Did some more PCB design and added some datasheets
Parts:
- added C1, C2: 0.1uF, rcl:C-USC0805
- added C3, C4: 10uF, rcl:C-USC0805
- added SV1: (no value), con-lstb:MA05-1
Connections:
- new net AC: SV1.2
- new net FAN: SV1.1
- new net HEAT: SV1.3
- net GND: now also C1.2, C2.2, C3.2, C4.2, SV1.4
- net VCC: now also C1.1, C2.1, C3.1, C4.1, SV1.5
Changed lines of the file:
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@@
 <?xml version="1.0" encoding="utf-8"?>
 <!DOCTYPE eagle SYSTEM "eagle.dtd">
-<eagle version="6.2">
+<eagle version="6.1">
 <drawing>
 <settings>
@@
 <layers>
 <layer number="1" name="Top" color="4" fill="1" visible="no" active="no"/>
+<layer number="2" name="Route2" color="1" fill="3" visible="no" active="no"/>
+<layer number="3" name="Route3" color="4" fill="3" visible="no" active="no"/>
+<layer number="4" name="Route4" color="1" fill="4" visible="no" active="no"/>
+<layer number="5" name="Route5" color="4" fill="4" visible="no" active="no"/>
+<layer number="6" name="Route6" color="1" fill="8" visible="no" active="no"/>
+<layer number="7" name="Route7" color="4" fill="8" visible="no" active="no"/>
+<layer number="8" name="Route8" color="1" fill="2" visible="no" active="no"/>
+<layer number="9" name="Route9" color="4" fill="2" visible="no" active="no"/>
+<layer number="10" name="Route10" color="1" fill="7" visible="no" active="no"/>
+<layer number="11" name="Route11" color="4" fill="7" visible="no" active="no"/>
+<layer number="12" name="Route12" color="1" fill="5" visible="no" active="no"/>
+<layer number="13" name="Route13" color="4" fill="5" visible="no" active="no"/>
+<layer number="14" name="Route14" color="1" fill="6" visible="no" active="no"/>
+<layer number="15" name="Route15" color="4" fill="6" visible="no" active="no"/>
 <layer number="16" name="Bottom" color="1" fill="1" visible="no" active="no"/>
 <layer number="17" name="Pads" color="2" fill="1" visible="no" active="no"/>
@@
 <part name="SUPPLY2" library="supply2" deviceset="VCC" device=""/>
 <part name="GND3" library="supply1" deviceset="GND" device=""/>
+<part name="SV1" library="con-lstb" deviceset="MA05-1" device=""/>
+<part name="C1" library="rcl" deviceset="C-US" device="C0805" value="0.1uF"/>
+<part name="C2" library="rcl" deviceset="C-US" device="C0805" value="0.1uF"/>
+<part name="C3" library="rcl" deviceset="C-US" device="C0805" value="10uF"/>
+<part name="C4" library="rcl" deviceset="C-US" device="C0805" value="10uF"/>
+<part name="SUPPLY3" library="supply2" deviceset="VCC" device=""/>
+<part name="GND4" library="supply1" deviceset="GND" device=""/>
 </parts>
 <sheets>
@@
 <instance part="SUPPLY2" gate="G$1" x="88.9" y="81.28"/>
 <instance part="GND3" gate="1" x="88.9" y="58.42"/>
+<instance part="SV1" gate="G$1" x="137.16" y="96.52"/>
+<instance part="C1" gate="G$1" x="38.1" y="104.14"/>
+<instance part="C2" gate="G$1" x="48.26" y="104.14"/>
+<instance part="C3" gate="G$1" x="58.42" y="104.14"/>
+<instance part="C4" gate="G$1" x="68.58" y="104.14"/>
+<instance part="SUPPLY3" gate="G$1" x="38.1" y="109.22"/>
+<instance part="GND4" gate="1" x="38.1" y="96.52"/>
 </instances>
 <busses>
@@
 <pinref part="SUPPLY2" gate="G$1" pin="VCC"/>
 <wire x1="88.9" y1="68.58" x2="88.9" y2="78.74" width="0.1524" layer="91"/>
+</segment>
+<segment>
+<pinref part="SV1" gate="G$1" pin="5"/>
+<wire x1="144.78" y1="101.6" x2="147.32" y2="101.6" width="0.1524" layer="91"/>
+<label x="144.78" y="101.6" size="1.778" layer="95"/>
+</segment>
+<segment>
+<pinref part="C1" gate="G$1" pin="1"/>
+<pinref part="C4" gate="G$1" pin="1"/>
+<wire x1="38.1" y1="106.68" x2="48.26" y2="106.68" width="0.1524" layer="91"/>
+<pinref part="SUPPLY3" gate="G$1" pin="VCC"/>
+<junction x="38.1" y="106.68"/>
+<pinref part="C2" gate="G$1" pin="1"/>
+<junction x="48.26" y="106.68"/>
+<wire x1="48.26" y1="106.68" x2="58.42" y2="106.68" width="0.1524" layer="91"/>
+<pinref part="C3" gate="G$1" pin="1"/>
+<junction x="58.42" y="106.68"/>
+<wire x1="58.42" y1="106.68" x2="68.58" y2="106.68" width="0.1524" layer="91"/>
+<junction x="68.58" y="106.68"/>
 </segment>
 </net>
@@
 <wire x1="88.9" y1="63.5" x2="88.9" y2="60.96" width="0.1524" layer="91"/>
 </segment>
+<segment>
+<pinref part="SV1" gate="G$1" pin="4"/>
+<wire x1="144.78" y1="99.06" x2="147.32" y2="99.06" width="0.1524" layer="91"/>
+<label x="144.78" y="99.06" size="1.778" layer="95"/>
+</segment>
+<segment>
+<pinref part="C1" gate="G$1" pin="2"/>
+<pinref part="C4" gate="G$1" pin="2"/>
+<wire x1="38.1" y1="99.06" x2="48.26" y2="99.06" width="0.1524" layer="91"/>
+<pinref part="GND4" gate="1" pin="GND"/>
+<junction x="38.1" y="99.06"/>
+<pinref part="C2" gate="G$1" pin="2"/>
+<junction x="48.26" y="99.06"/>
+<wire x1="48.26" y1="99.06" x2="58.42" y2="99.06" width="0.1524" layer="91"/>
+<pinref part="C3" gate="G$1" pin="2"/>
+<junction x="58.42" y="99.06"/>
+<wire x1="58.42" y1="99.06" x2="68.58" y2="99.06" width="0.1524" layer="91"/>
+<junction x="68.58" y="99.06"/>
+</segment>
 </net>
 <net name="RESET" class="0">
@@
 </segment>
 </net>
+<net name="HEAT" class="0">
+<segment>
+<pinref part="SV1" gate="G$1" pin="3"/>
+<wire x1="144.78" y1="96.52" x2="147.32" y2="96.52" width="0.1524" layer="91"/>
+<label x="144.78" y="96.52" size="1.778" layer="95"/>
+</segment>
+</net>
+<net name="AC" class="0">
+<segment>
+<pinref part="SV1" gate="G$1" pin="2"/>
+<wire x1="144.78" y1="93.98" x2="147.32" y2="93.98" width="0.1524" layer="91"/>
+<label x="144.78" y="93.98" size="1.778" layer="95"/>
+</segment>
+</net>
+<net name="FAN" class="0">
+<segment>
+<pinref part="SV1" gate="G$1" pin="1"/>
+<wire x1="144.78" y1="91.44" x2="147.32" y2="91.44" width="0.1524" layer="91"/>
+<label x="144.78" y="91.44" size="1.778" layer="95"/>
+</segment>
+</net>

Commit message: split into three boards and choose new mcu
Parts:
- removed MSP430F1232: F12X2---DW28, TI_MSP430_v16:F12X2---DW28
- added D1, D2, D3: 1N4148DO35-7, diode:1N4148DO35-7
- added JP1: (no value), pinhead:PINHD-1X4
- added K1, K2, K3: G5LE, relay:G5LE
- added T1, T2, T3: (no value), transistor-neu-to92:2N4401-NPN-TO92-EBC
- added U$1: F21X2---RHB32, TI_MSP430_v16:F21X2---RHB32
Connections:
- new net 5V+: D1.C, D2.C, D3.C, K11.1, K21.1, K31.1
- new net G: K32.S
- new net N$2: D1.A, K31.2, T1.C
- new net N$3: D2.A, K21.2, T2.C
- new net N$5: D3.A, K11.2, T3.C
- new net N$6: K12.O
- new net N$7: K22.O
- new net N$8: K32.O
- new net RST: JP1.4, U$1.5
- new net TEST: JP1.3, U$1.29
- new net VAC+: K12.P, K22.P, K32.P
- new net W: K12.S
- new net Y: K22.S
- net AC: now also T2.B, U$1.7
- net FAN: now also T1.B, U$1.8
- net GND: now also JP1.2, T1.E, T2.E, T3.E, U$1.1, U$1.33; no longer MSP430F1232.4
- net HEAT: now also T3.B, U$1.6
- net RN-RX: now also U$1.13; no longer MSP430F1232.15
- net RN-TX: now also U$1.14; no longer MSP430F1232.16
- net VCC: now also JP1.1, U$1.30; no longer MSP430F1232.2
Other:
- note added: "5V+"
- note added: "G"
- note added: "W"
- note added: "Y"

Commit message: removed relays from control
Parts:
- removed D1, D2, D3: 1N4148DO35-7, diode:1N4148DO35-7
- removed K1, K2, K3: G5LE, relay:G5LE
- removed T1, T2, T3: (no value), transistor-neu-to92:2N4401-NPN-TO92-EBC
Connections:
- removed net 5V+: D1.C, D2.C, D3.C, K11.1, K21.1, K31.1
- removed net G: K32.S
- removed net N$2: D1.A, K31.2, T1.C
- removed net N$3: D2.A, K21.2, T2.C
- removed net N$5: D3.A, K11.2, T3.C
- removed net N$6: K12.O
- removed net N$7: K22.O
- removed net N$8: K32.O
- removed net VAC+: K12.P, K22.P, K32.P
- removed net W: K12.S
- removed net Y: K22.S
- net AC: no longer T2.B
- net FAN: no longer T1.B
- net GND: no longer T1.E, T2.E, T3.E
- net HEAT: no longer T3.B
Other:
- note removed: "5V+"
- note removed: "G"
- note removed: "W"
- note removed: "Y"
Changed lines of the file:
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@@
 <part name="SUPPLY4" library="supply2" deviceset="VCC" device=""/>
 <part name="JP1" library="pinhead" deviceset="PINHD-1X4" device=""/>
-<part name="K1" library="relay" deviceset="G5LE" device=""/>
-<part name="K2" library="relay" deviceset="G5LE" device=""/>
-<part name="K3" library="relay" deviceset="G5LE" device=""/>
-<part name="D1" library="diode" deviceset="1N4148" device="DO35-7"/>
-<part name="D2" library="diode" deviceset="1N4148" device="DO35-7"/>
-<part name="D3" library="diode" deviceset="1N4148" device="DO35-7"/>
-<part name="T1" library="transistor-neu-to92" deviceset="*-NPN-" device="TO92-EBC" technology="2N4401"/>
-<part name="T2" library="transistor-neu-to92" deviceset="*-NPN-" device="TO92-EBC" technology="2N4401"/>
-<part name="T3" library="transistor-neu-to92" deviceset="*-NPN-" device="TO92-EBC" technology="2N4401"/>
-<part name="GND3" library="supply1" deviceset="GND" device=""/>
-<part name="GND6" library="supply1" deviceset="GND" device=""/>
-<part name="GND7" library="supply1" deviceset="GND" device=""/>
 </parts>
 <sheets>
@@
 <net name="RN-RX" class="0">
 <segment>
-<wire x1="33.02" y1="60.96" x2="22.86" y2="60.96" width="0.1524" layer="91"/>
+<wire x1="33.02" y1="60.96" x2="25.4" y2="60.96" width="0.1524" layer="91"/>
 <pinref part="RN-131C" gate="G$1" pin="RX"/>
+<junction x="25.4" y="60.96"/>
 </segment>
 <segment>
@@
 <net name="RN-TX" class="0">
 <segment>
-<wire x1="33.02" y1="58.42" x2="22.86" y2="58.42" width="0.1524" layer="91"/>
+<wire x1="33.02" y1="58.42" x2="25.4" y2="58.42" width="0.1524" layer="91"/>
 <pinref part="RN-131C" gate="G$1" pin="TX"/>
+<junction x="25.4" y="58.42"/>
 </segment>
 <segment>
@@
 <net name="RESET" class="0">
 <segment>
-<wire x1="71.12" y1="66.04" x2="78.74" y2="66.04" width="0.1524" layer="91"/>
+<wire x1="71.12" y1="66.04" x2="76.2" y2="66.04" width="0.1524" layer="91"/>
 <pinref part="RN-131C" gate="G$1" pin="RESET"/>
+<junction x="76.2" y="66.04"/>
 </segment>
 </net>
@@
 </segment>
 </net>
-</nets>
-</sheet>
-<sheet>
-<plain>
-<text x="25.4" y="27.94" size="1.778" layer="91">5V+</text>
-<text x="45.72" y="27.94" size="1.778" layer="91">5V+</text>
-<text x="5.08" y="27.94" size="1.778" layer="91">5V+</text>
-<text x="60.706" y="16.002" size="1.778" layer="95">W</text>
-<text x="73.914" y="16.002" size="1.778" layer="95">Y</text>
-<text x="86.614" y="16.002" size="1.778" layer="95">G</text>
-</plain>
-<instances>
-<instance part="K1" gate="1" x="10.16" y="20.32"/>
-<instance part="K1" gate="2" x="66.04" y="5.08"/>
-<instance part="K2" gate="1" x="30.48" y="20.32"/>
-<instance part="K2" gate="2" x="78.74" y="5.08"/>
-<instance part="K3" gate="1" x="50.8" y="20.32"/>
-<instance part="K3" gate="2" x="91.44" y="5.08"/>
-<instance part="D1" gate="G$1" x="43.18" y="20.32" smashed="yes" rot="R90">
-<attribute name="NAME" x="42.6974" y="22.86" size="1.778" layer="95" rot="R90"/>
-</instance>
-<instance part="D2" gate="G$1" x="22.86" y="20.32" smashed="yes" rot="R90">
-<attribute name="NAME" x="22.3774" y="22.86" size="1.778" layer="95" rot="R90"/>
-</instance>
-<instance part="D3" gate="G$1" x="2.54" y="20.32" smashed="yes" rot="R90">
-<attribute name="NAME" x="2.0574" y="22.86" size="1.778" layer="95" rot="R90"/>
-</instance>
-<instance part="T1" gate="G$1" x="48.26" y="10.16"/>
-<instance part="T2" gate="G$1" x="27.94" y="10.16"/>
-<instance part="T3" gate="G$1" x="7.62" y="10.16"/>
-<instance part="GND3" gate="1" x="50.8" y="2.54"/>
-<instance part="GND6" gate="1" x="30.48" y="2.54"/>
-<instance part="GND7" gate="1" x="10.16" y="2.54"/>
-</instances>
-<busses>
-</busses>
-<nets>
-<net name="N$2" class="0">
-<segment>
-<pinref part="D1" gate="G$1" pin="A"/>
-<wire x1="43.18" y1="17.78" x2="43.18" y2="15.24" width="0.1524" layer="91"/>
-<pinref part="K3" gate="1" pin="2"/>
-<wire x1="43.18" y1="15.24" x2="50.8" y2="15.24" width="0.1524" layer="91"/>
-<pinref part="T1" gate="G$1" pin="C"/>
-<junction x="50.8" y="15.24"/>
-</segment>
-</net>
-<net name="N$3" class="0">
-<segment>
-<pinref part="K2" gate="1" pin="2"/>
-<wire x1="30.48" y1="15.24" x2="22.86" y2="15.24" width="0.1524" layer="91"/>
-<pinref part="D2" gate="G$1" pin="A"/>
-<wire x1="22.86" y1="15.24" x2="22.86" y2="17.78" width="0.1524" layer="91"/>
-<pinref part="T2" gate="G$1" pin="C"/>
-<junction x="30.48" y="15.24"/>
-</segment>
-</net>
-<net name="N$5" class="0">
-<segment>
-<pinref part="K1" gate="1" pin="2"/>
-<wire x1="10.16" y1="15.24" x2="2.54" y2="15.24" width="0.1524" layer="91"/>
-<pinref part="D3" gate="G$1" pin="A"/>
-<wire x1="2.54" y1="15.24" x2="2.54" y2="17.78" width="0.1524" layer="91"/>
-<pinref part="T3" gate="G$1" pin="C"/>
-<junction x="10.16" y="15.24"/>
-</segment>
-</net>
-<net name="GND" class="0">
-<segment>
-<pinref part="T1" gate="G$1" pin="E"/>
-<pinref part="GND3" gate="1" pin="GND"/>
-</segment>
-<segment>
-<pinref part="T2" gate="G$1" pin="E"/>
-<pinref part="GND6" gate="1" pin="GND"/>
-</segment>
-<segment>
-<pinref part="T3" gate="G$1" pin="E"/>
-<pinref part="GND7" gate="1" pin="GND"/>
-</segment>
-</net>
-<net name="VAC+" class="0">
-<segment>
-<pinref part="K1" gate="2" pin="P"/>
-<pinref part="K3" gate="2" pin="P"/>
-<wire x1="66.04" y1="2.54" x2="78.74" y2="2.54" width="0.1524" layer="91"/>
-<junction x="66.04" y="2.54"/>
-<pinref part="K2" gate="2" pin="P"/>
-<junction x="78.74" y="2.54"/>
-<wire x1="78.74" y1="2.54" x2="91.44" y2="2.54" width="0.1524" layer="91"/>
-<junction x="91.44" y="2.54"/>
-</segment>
-</net>
-<net name="5V+" class="0">
-<segment>
-<pinref part="D2" gate="G$1" pin="C"/>
-<wire x1="22.86" y1="22.86" x2="22.86" y2="25.4" width="0.1524" layer="91"/>
-<pinref part="K2" gate="1" pin="1"/>
-<wire x1="22.86" y1="25.4" x2="30.48" y2="25.4" width="0.1524" layer="91"/>
-<wire x1="30.48" y1="25.4" x2="30.48" y2="27.94" width="0.1524" layer="91"/>
-<junction x="30.48" y="27.94"/>
-</segment>
-<segment>
-<pinref part="D3" gate="G$1" pin="C"/>
-<wire x1="2.54" y1="22.86" x2="2.54" y2="25.4" width="0.1524" layer="91"/>
-<pinref part="K1" gate="1" pin="1"/>
-<wire x1="2.54" y1="25.4" x2="10.16" y2="25.4" width="0.1524" layer="91"/>
-<wire x1="10.16" y1="25.4" x2="10.16" y2="27.94" width="0.1524" layer="91"/>
-<junction x="10.16" y="27.94"/>
-</segment>
-<segment>
-<pinref part="K3" gate="1" pin="1"/>
-<wire x1="50.8" y1="25.4" x2="43.18" y2="25.4" width="0.1524" layer="91"/>
-<pinref part="D1" gate="G$1" pin="C"/>
-<wire x1="43.18" y1="25.4" x2="43.18" y2="22.86" width="0.1524" layer="91"/>
-<wire x1="50.8" y1="25.4" x2="50.8" y2="27.94" width="0.1524" layer="91"/>
-<junction x="50.8" y="27.94"/>
-</segment>
-</net>
-<net name="W" class="0">
-<segment>
-<wire x1="60.96" y1="10.16" x2="60.96" y2="15.24" width="0.1524" layer="91"/>
-<junction x="60.96" y="15.24"/>
-<wire x1="60.96" y1="10.16" x2="63.5" y2="10.16" width="0.1524" layer="91"/>
-<pinref part="K1" gate="2" pin="S"/>
-<junction x="60.96" y="10.16"/>
-<junction x="63.5" y="10.16"/>
-</segment>
-</net>
-<net name="Y" class="0">
-<segment>
-<wire x1="73.66" y1="10.16" x2="73.66" y2="15.24" width="0.1524" layer="91"/>
-<junction x="73.66" y="15.24"/>
-<wire x1="73.66" y1="10.16" x2="76.2" y2="10.16" width="0.1524" layer="91"/>
-<pinref part="K2" gate="2" pin="S"/>
-<junction x="73.66" y="10.16"/>
-<junction x="76.2" y="10.16"/>
-</segment>
-</net>
-<net name="G" class="0">
-<segment>
-<wire x1="86.36" y1="10.16" x2="86.36" y2="15.24" width="0.1524" layer="91"/>
-<junction x="86.36" y="15.24"/>
-<wire x1="86.36" y1="10.16" x2="88.9" y2="10.16" width="0.1524" layer="91"/>
-<pinref part="K3" gate="2" pin="S"/>
-<junction x="86.36" y="10.16"/>
-<junction x="88.9" y="10.16"/>
-</segment>
-</net>
-<net name="HEAT" class="0">
-<segment>
-<pinref part="T3" gate="G$1" pin="B"/>
-<wire x1="5.08" y1="10.16" x2="2.54" y2="10.16" width="0.1524" layer="91"/>
-<junction x="2.54" y="10.16"/>
-<label x="0" y="7.62" size="1.778" layer="95"/>
-</segment>
-</net>
-<net name="FAN" class="0">
-<segment>
-<pinref part="T1" gate="G$1" pin="B"/>
-<wire x1="45.72" y1="10.16" x2="43.18" y2="10.16" width="0.1524" layer="91"/>
-<junction x="43.18" y="10.16"/>
-<label x="43.18" y="7.62" size="1.778" layer="95"/>
-</segment>
-</net>
-<net name="AC" class="0">
-<segment>
-<pinref part="T2" gate="G$1" pin="B"/>
-<wire x1="25.4" y1="10.16" x2="22.86" y2="10.16" width="0.1524" layer="91"/>
-<junction x="22.86" y="10.16"/>
-<label x="22.86" y="7.62" size="1.778" layer="95"/>
-</segment>
-</net>
-<net name="N$6" class="0">
-<segment>
-<pinref part="K1" gate="2" pin="O"/>
-<wire x1="68.58" y1="10.16" x2="71.12" y2="10.16" width="0.1524" layer="91"/>
-</segment>
-</net>
-<net name="N$7" class="0">
-<segment>
-<pinref part="K2" gate="2" pin="O"/>
-<wire x1="81.28" y1="10.16" x2="83.82" y2="10.16" width="0.1524" layer="91"/>
-</segment>
-</net>
-<net name="N$8" class="0">
-<segment>
-<pinref part="K3" gate="2" pin="O"/>
-<wire x1="93.98" y1="10.16" x2="96.52" y2="10.16" width="0.1524" layer="91"/>
-</segment>
-</net>
