File: eagle_design/Control.sch (EAGLE design)
At the start: 17 parts

Commit message: finished control board
Parts:
- added SW1: EC12E_SW, switch-alps:EC12E_SW
Connections:
- removed net P2_2: U$1.12
- removed net P2_3: U$1.16
- removed net P2_4: U$1.17
- removed net P3_2: U$1.13
- removed net P3_3: U$1.14
- removed net P3_4: U$1.15
- new net A: SW1G$1.B, U$1.13
- new net B: SW1G$1.A, U$1.14
- new net OFF: SW1G$2.2, U$1.12
- net AC: now also U$1.16
- net FAN: now also U$1.15
- net GND: now also SPW.4, SW1G$1.C; no longer SPW.3
- net HEAT: now also U$1.17
- net RST: now also SPW.3; no longer SPW.4
- net TEST: now also SPW.1; no longer SPW.2
- net VCC: now also SPW.2, SW1G$2.1; no longer SPW.1
Changed lines of the file:
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@@
 <part name="R1" library="Panasonic_By_element14_Batch_1" deviceset="ERA-3AEB104V" device="" value="100 kOhm"/>
 <part name="U$3" library="TylersLib" deviceset="NHD-C12832A1Z-FSW-FBW-3V3" device=""/>
+<part name="SW1" library="switch-alps" deviceset="EC12E_SW" device=""/>
 </parts>
 <sheets>
@@
 <instance part="R1" gate="A" x="127" y="10.16"/>
 <instance part="U$3" gate="G$1" x="172.72" y="22.86"/>
+<instance part="SW1" gate="G$1" x="99.06" y="73.66"/>
+<instance part="SW1" gate="G$2" x="83.82" y="74.93"/>
 </instances>
 <busses>
@@
 </segment>
 <segment>
-<pinref part="SPW" gate="A" pin="1"/>
-<wire x1="40.64" y1="60.96" x2="33.02" y2="60.96" width="0.1524" layer="91"/>
-<label x="33.02" y="60.96" size="1.778" layer="95"/>
-<junction x="33.02" y="60.96"/>
-</segment>
-<segment>
 <pinref part="U$1" gate="G$1" pin="1"/>
 <wire x1="6.35" y1="38.1" x2="2.54" y2="38.1" width="0.1524" layer="91"/>
@@
 <label x="134.62" y="27.94" size="1.778" layer="95"/>
 </segment>
+<segment>
+<pinref part="SW1" gate="G$2" pin="1"/>
+<wire x1="88.9" y1="74.93" x2="90.678" y2="74.93" width="0.1524" layer="91"/>
+<junction x="90.678" y="74.93"/>
+</segment>
+<segment>
+<pinref part="SPW" gate="A" pin="2"/>
+<wire x1="48.26" y1="60.96" x2="53.34" y2="60.96" width="0.1524" layer="91"/>
+<junction x="53.34" y="60.96"/>
+<label x="53.34" y="60.96" size="1.778" layer="95"/>
+</segment>
 </net>
 <net name="GND" class="0">
@@
 <junction x="7.62" y="55.88"/>
 <pinref part="C2" gate="G$1" pin="2"/>
-</segment>
-<segment>
-<pinref part="SPW" gate="A" pin="3"/>
-<wire x1="40.64" y1="58.42" x2="33.02" y2="58.42" width="0.1524" layer="91"/>
-<label x="33.02" y="58.42" size="1.778" layer="95"/>
-<junction x="33.02" y="58.42"/>
 </segment>
 <segment>
@@
 <label x="129.54" y="33.02" size="1.778" layer="95"/>
 </segment>
+<segment>
+<pinref part="SW1" gate="G$1" pin="C"/>
+<wire x1="99.06" y1="71.12" x2="99.06" y2="68.58" width="0.1524" layer="91"/>
+<junction x="99.06" y="68.58"/>
+</segment>
+<segment>
+<pinref part="SPW" gate="A" pin="4"/>
+<wire x1="48.26" y1="58.42" x2="53.34" y2="58.42" width="0.1524" layer="91"/>
+<junction x="53.34" y="58.42"/>
+<label x="53.34" y="58.42" size="1.778" layer="95"/>
+</segment>
 </net>
 <net name="TEST" class="0">
-<segment>
-<pinref part="SPW" gate="A" pin="2"/>
-<wire x1="48.26" y1="60.96" x2="55.88" y2="60.96" width="0.1524" layer="91"/>
-<label x="53.34" y="60.96" size="1.778" layer="95"/>
-<junction x="55.88" y="60.96"/>
-</segment>
 <segment>
 <pinref part="U$1" gate="G$1" pin="25"/>
@@
 <label x="58.42" y="30.48" size="1.778" layer="95"/>
 </segment>
+<segment>
+<pinref part="SPW" gate="A" pin="1"/>
+<wire x1="40.64" y1="60.96" x2="35.56" y2="60.96" width="0.1524" layer="91"/>
+<junction x="35.56" y="60.96"/>
+<label x="30.48" y="60.96" size="1.778" layer="95"/>
+</segment>
 </net>
 <net name="RST" class="0">
-<segment>
-<pinref part="SPW" gate="A" pin="4"/>
-<wire x1="48.26" y1="58.42" x2="55.88" y2="58.42" width="0.1524" layer="91"/>
-<label x="53.34" y="58.42" size="1.778" layer="95"/>
-<junction x="55.88" y="58.42"/>
-</segment>
 <segment>
 <pinref part="U$1" gate="G$1" pin="24"/>
@@
 <label x="58.42" y="27.94" size="1.778" layer="95"/>
 </segment>
-</net>
-<net name="P3_3" class="0">
-<segment>
-<pinref part="U$1" gate="G$1" pin="14"/>
-<wire x1="6.35" y1="5.08" x2="2.54" y2="5.08" width="0.1524" layer="91"/>
-<junction x="2.54" y="5.08"/>
-</segment>
-</net>
-<net name="P3_2" class="0">
-<segment>
-<pinref part="U$1" gate="G$1" pin="13"/>
-<wire x1="6.35" y1="7.62" x2="2.54" y2="7.62" width="0.1524" layer="91"/>
-<junction x="2.54" y="7.62"/>
+<segment>
+<pinref part="SPW" gate="A" pin="3"/>
+<wire x1="40.64" y1="58.42" x2="35.56" y2="58.42" width="0.1524" layer="91"/>
+<junction x="35.56" y="58.42"/>
+<label x="30.48" y="58.42" size="1.778" layer="95"/>
 </segment>
 </net>
@@
 </segment>
 </net>
-<net name="P2_2" class="0">
-<segment>
-<pinref part="U$1" gate="G$1" pin="12"/>
-<wire x1="6.35" y1="10.16" x2="2.54" y2="10.16" width="0.1524" layer="91"/>
-<junction x="2.54" y="10.16"/>
-</segment>
-</net>
 <net name="P2_1" class="0">
 <segment>
@@
 </segment>
 </net>
-<net name="P2_4" class="0">
-<segment>
-<pinref part="U$1" gate="G$1" pin="17"/>
-<wire x1="53.34" y1="10.16" x2="58.42" y2="10.16" width="0.1524" layer="91"/>
-<junction x="58.42" y="10.16"/>
-</segment>
-</net>
-<net name="P2_3" class="0">
-<segment>
-<pinref part="U$1" gate="G$1" pin="16"/>
-<wire x1="53.34" y1="7.62" x2="58.42" y2="7.62" width="0.1524" layer="91"/>
-<junction x="58.42" y="7.62"/>
-</segment>
-</net>
 <net name="P3_7" class="0">
 <segment>
@@
 <wire x1="53.34" y1="15.24" x2="58.42" y2="15.24" width="0.1524" layer="91"/>
 <junction x="58.42" y="15.24"/>
-</segment>
-</net>
-<net name="P3_4" class="0">
-<segment>
-<pinref part="U$1" gate="G$1" pin="15"/>
-<wire x1="53.34" y1="5.08" x2="58.42" y2="5.08" width="0.1524" layer="91"/>
-<junction x="58.42" y="5.08"/>
 </segment>
 </net>
@@
 <label x="66.04" y="50.8" size="1.778" layer="95"/>
 </segment>
+<segment>
+<pinref part="U$1" gate="G$1" pin="15"/>
+<wire x1="53.34" y1="5.08" x2="58.42" y2="5.08" width="0.1524" layer="91"/>
+<junction x="58.42" y="5.08"/>
+<label x="58.42" y="5.08" size="1.778" layer="95"/>
+</segment>
 </net>
 <net name="AC" class="0">
@@
 <label x="66.04" y="48.26" size="1.778" layer="95"/>
 </segment>
+<segment>
+<pinref part="U$1" gate="G$1" pin="16"/>
+<wire x1="53.34" y1="7.62" x2="58.42" y2="7.62" width="0.1524" layer="91"/>
+<junction x="58.42" y="7.62"/>
+<label x="58.42" y="7.62" size="1.778" layer="95"/>
+</segment>
 </net>
 <net name="HEAT" class="0">
@@
 <junction x="68.58" y="45.72"/>
 <label x="66.04" y="45.72" size="1.778" layer="95"/>
+</segment>
+<segment>
+<pinref part="U$1" gate="G$1" pin="17"/>
+<wire x1="53.34" y1="10.16" x2="58.42" y2="10.16" width="0.1524" layer="91"/>
+<junction x="58.42" y="10.16"/>
+<label x="58.42" y="10.16" size="1.778" layer="95"/>
 </segment>
 </net>
@@
 </segment>
 </net>
+<net name="OFF" class="0">
+<segment>
+<pinref part="SW1" gate="G$2" pin="2"/>
+<wire x1="78.74" y1="74.93" x2="76.454" y2="74.93" width="0.1524" layer="91"/>
+<junction x="76.454" y="74.93"/>
+</segment>
+<segment>
+<pinref part="U$1" gate="G$1" pin="12"/>
+<wire x1="6.35" y1="10.16" x2="2.54" y2="10.16" width="0.1524" layer="91"/>
+<junction x="2.54" y="10.16"/>
+<label x="-2.54" y="10.16" size="1.778" layer="95"/>
+</segment>
+</net>
+<net name="B" class="0">
+<segment>
+<pinref part="SW1" gate="G$1" pin="A"/>
+<wire x1="96.52" y1="81.28" x2="96.52" y2="83.82" width="0.1524" layer="91"/>
+<junction x="96.52" y="83.82"/>
+</segment>
+<segment>
+<pinref part="U$1" gate="G$1" pin="14"/>
+<wire x1="6.35" y1="5.08" x2="2.54" y2="5.08" width="0.1524" layer="91"/>
+<junction x="2.54" y="5.08"/>
+<label x="-2.54" y="5.08" size="1.778" layer="95"/>
+</segment>
+</net>
+<net name="A" class="0">
+<segment>
+<pinref part="SW1" gate="G$1" pin="B"/>
+<wire x1="101.6" y1="81.28" x2="101.6" y2="83.82" width="0.1524" layer="91"/>
+<junction x="101.6" y="83.82"/>
+</segment>
+<segment>
+<pinref part="U$1" gate="G$1" pin="13"/>
+<wire x1="6.35" y1="7.62" x2="2.54" y2="7.62" width="0.1524" layer="91"/>
+<junction x="2.54" y="7.62"/>
+<label x="-2.54" y="7.62" size="1.778" layer="95"/>
+</segment>
+</net>
